Commit message: aruco recognition

File: ros2_iiwa/iiwa_description/urdf/camera.xacro (robot description, xacro)
@@ -18,5 +18,5 @@
         <parent link="${prefix}tool0"/>
         <child link="${prefix}camera_link"/>
-        <origin xyz="0 0 0.01" rpy="0 -1.57 -1.57"/>
+        <origin xyz="0 0 0.01" rpy="0 -1.57 -3.14"/>
       </joint>
       <gazebo reference="camera_link">

Commit message: fix orientation errors

File: ros2_iiwa/iiwa_description/urdf/camera.xacro (robot description, xacro)
@@ -7,5 +7,5 @@
         <visual>
           <geometry>
-            <box size="0.02 0.02 0.02"/>
+            <box size="0.01 0.01 0.01"/>
           </geometry>
           <material name="camera_material"> <!-- Add the name attribute here -->
@@ -13,10 +13,10 @@
           </material>
         </visual>
-        <origin xyz="0 0 0.01" rpy="0 0 0"/>
+        <origin xyz="0 0 0" rpy="0 0 0"/>
       </link>
       <joint name="camera_joint" type="fixed">
         <parent link="${prefix}tool0"/>
         <child link="${prefix}camera_link"/>
-        <origin xyz="0 0 0.01" rpy="0 -1.57 -3.14"/>
+        <origin xyz="0 0 0" rpy="0 -1.57 -3.14"/>
       </joint>
       <gazebo reference="camera_link">

Commit message: fix orientation + torques controllers

File: ros2_iiwa/iiwa_description/urdf/camera.xacro (robot description, xacro)
@@ -18,5 +18,6 @@
         <parent link="${prefix}tool0"/>
         <child link="${prefix}camera_link"/>
-        <origin xyz="0 0 0" rpy="0 -1.57 -3.14"/>
+        <axis xyz="0 1 0"/>
+        <origin xyz="0 0 0" rpy="0 -1.57 3.14"/>
       </joint>
       <gazebo reference="camera_link">

Commit message: modified readme

File: ros2_iiwa/iiwa_description/urdf/camera.xacro (robot description, xacro)
@@ -4,4 +4,10 @@
     <!-- Optional Camera -->
     <xacro:if value="${use_vision}">
+      <joint name="camera_joint" type="fixed">
+        <parent link="${prefix}tool0"/>
+        <child link="${prefix}camera_link"/>
+        <axis xyz="0 1 0"/>
+        <origin xyz="0 0 0" rpy="0 -1.57 3.14"/>
+      </joint>
       <link name="${prefix}camera_link">
         <visual>
@@ -15,10 +21,10 @@
         <origin xyz="0 0 0" rpy="0 0 0"/>
       </link>
-      <joint name="camera_joint" type="fixed">
-        <parent link="${prefix}tool0"/>
-        <child link="${prefix}camera_link"/>
-        <axis xyz="0 1 0"/>
-        <origin xyz="0 0 0" rpy="0 -1.57 3.14"/>
+      <joint name="camera_optical_joint" type="fixed">
+          <parent link="${prefix}camera_link"/>
+          <child link="camera_link_optical"/>
+          <origin xyz="0 0 0" rpy="-1.57 0 -1.57"/>
       </joint>
+      <link name="camera_link_optical"></link>
       <gazebo reference="camera_link">
           <sensor name="camera" type="camera">
